File: Pegasus_Servo_Interface_V1/Pegasus_Servo_Interface_V1.kicad_pcb (KiCad board)
At the start: 2 copper layers, 32 x 61.5 mm, 14 parts, among them J1 RJ45_Shielded, J2 Pos_Feedback, J3 DE9_Receptacle_MountingHoles, U1 XC6220B331MR, U2 SN65LVDS2D

Commit message: Add files via upload
Parts:
- added LOGO1: teTra, Symbol:teTra-LOGO, F.Cu at (153.1, 108.2)
- J1: value RJ45_Shielded -> RJ45
- U1: value XC6220B331MR -> XC6216D332PR-G
Other:
- board text added: "2024/07/03 Pegasus_Servo_Interface_V1"

Commit message: Add files via upload
Parts:
- removed H1: BAT+, MountingHole:MountingHole_3.2mm_M3_DIN965_Pad_TopBottom
- removed H2: BAT-, MountingHole:MountingHole_3.2mm_M3_DIN965_Pad_TopBottom
- added J4: Molex 5569, Connector_Molex:Molex_Mini-Fit_Jr_5569-04A2_2x02_P4.20mm_Horizontal, F.Cu at (154.6, 107.7)
- moved LOGO1 11.6 mm to (142.2, 104.3)
- moved C5 5.97 mm to (147.9, 100.1)
Routing:
- net /+UB: track 33.8 -> 29.6 mm
- net /PWM_TTL: track 31.6 -> 32.9 mm
- net GND: vias 84 -> 86
Other:
- board text added: "2024/07/03 Servo_Interface_V1"
- board text added: "B+"
- board text added: "B-"
- board text removed: "2024/07/03 Pegasus_Servo_Interface_V1"
